Commit message: Enhance simulation: Format URDF, fix arm visuals, add 3x3 grid autonomy script, and add teleop obstacles (transformer, barrel, concrete block)

File: src/solar_rover_description/urdf/rover.urdf (robot description, URDF)
Before this commit: robot solar_rover_pro, 13 links, 12 joints
Links:
- link arm_base: mass 1.0 -> 0.1; geometry collision cylinder length=0.001 radius=0.001; visual mesh filename=file:///home/sam_k/ros2_sam/src/solar_rover_description/mes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 scale=0.012 0.012 0.012
- link arm_lower: mass 1.0 -> 0.1; geometry collision cylinder length=0.001 radius=0.001; visual mesh filename=file:///home/sam_k/ros2_sam/src/solar_rover_description/mes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 scale=0.012 0.012 0.012
- link arm_upper: mass 1.0 -> 0.1; geometry collision cylinder length=0.001 radius=0.001; visual mesh filename=file:///home/sam_k/ros2_sam/src/solar_rover_description/mes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 scale=0.012 0.012 0.012
- link brush: mass 1.0 -> 0.1; geometry collision cylinder length=0.001 radius=0.001; visual mesh filename=file:///home/sam_k/ros2_sam/src/solar_rover_description/mes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 scale=0.012 0.012 0.012

Commit message: Fix LiDAR joint translation to align with rear sensor mast and integrate static suspension/mast meshes into base_link

File: src/solar_rover_description/urdf/rover.urdf (robot description, URDF)
Before this commit: robot solar_rover_pro, 13 links, 12 joints
Links:
- link base_link: geometry collision box size=1.2 0.4 0.2; visual mesh filename=file:///home/sam_k/ros2_sam/src/solar_rover_description/mes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 scale=0.012 0.012 0.012
Joints:
- joint lidar_joint: origin xyz=0.75 0 1.05 -> xyz=-0.45 0 1.25

Commit message: feat: added RViz visualization and implemented Gazebo Odometry

File: src/solar_rover_description/urdf/rover.urdf (robot description, URDF)
Before this commit: robot solar_rover_pro, 13 links, 12 joints
Joints:
- joint lidar_joint: origin xyz=-0.45 0 1.25 -> xyz=0.75 0 1.05
